Commit message: adicionando os modelos do carro corretamente

File: eufs_sim/eufs_racecar/robots/carro_enel/robot.urdf.xacro (robot description, xacro)
@@ -1 +1,60 @@
-/home/gustavo/eufs_sim_teste/eufs_sim/eufs_racecar/robots/carro_enel/robot.urdf.xacro
+<?xml version="1.0"?>
+<robot name="carro_enel" xmlns:xacro="http://www.ros.org/wiki/xacro">
+    <!-- ***************** -->
+    <!-- Config parameters -->
+    <!-- ***************** -->
+    <!--  Load the config file  -->
+    <xacro:property name="config" value="${load_yaml('$(arg config_file)')}"/>
+    <!-- ***************** -->
+    <!-- Global parameters -->
+    <!-- ***************** -->
+    <xacro:property name="PI" value="3.1415926535897931"/>
+    <!-- If the gazebo_ros_race_car_model should publish the ground truth tf -->
+    <xacro:arg name="publish_tf" default="false"/>
+    <!-- If the perception stack should be simulated or if sensors should be used -->
+    <xacro:arg name="simulate_perception" default="true"/>
+    <!-- ***************** -->
+    <!-- Imported elements -->
+    <!-- ***************** -->
+    <!--  Import the wheels  -->
+    <xacro:include filename="$(find eufs_racecar)/urdf/carro_enel_wheels.urdf.xacro"/>
+    <!-- Import EUFS base element with the chassis -->
+    <xacro:include filename="$(find eufs_racecar)/urdf/carro_enel_base.urdf.xacro" />
+    <!-- Import all available sensors -->
+    <xacro:include filename="$(find eufs_sensors)/urdf/all_sensors.urdf.xacro" />
+    <!--  Include the plugins  -->
+    <xacro:include filename="$(find eufs_plugins)/urdf/eufs_plugins.gazebo.xacro" />
+    <!-- *************** -->
+    <!-- Robots Elements -->
+    <!-- *************** -->
+    <!-- Chassis of the car -->
+    <xacro:carro_enel_base chassis_mesh="file://$(find eufs_racecar)/meshes/carro_enel.dae"/>
+    <!-- Wheels -->
+    <xacro:wheels chassis_width="1.6" wheelbase="1.580"/>
+    <!-- *********************************************** -->
+    <!--                 MAIN SENSORS                    -->
+    <!-- *********************************************** -->
+    <!--     LOCATIONS: (XYZ)
+    IMU: 0.0 0.0 0.170
+    GPS: -0.110 0.0 0.9
+    LIDAR: 1.700 0.0 -0.150
+    STEREO CAM: -0.110 0.0 0.800 -->
+    <xacro:sensor_imu parent="chassis" prefix="sbg_imu" topic_prefix="">
+        <origin xyz="0.0 0.0 0.0" rpy="0 0 0"/>
+    </xacro:sensor_imu>
+    <xacro:sensor_gps parent="chassis" prefix="gps">
+        <origin xyz="0.0 0.0 0.4" rpy="0 0 0"/>
+    </xacro:sensor_gps>
+    <xacro:VLP-16R parent="chassis" name="velodyne" topic="/velodyne_points" hz="10" active="$(arg simulate_perception)">
+        <origin xyz="-0.15 0.0 0.79" rpy="0 ${1*M_PI/180.0} 0"/>
+    </xacro:VLP-16R>
+    <xacro:zed_camera parent="chassis" prefix="zed" active="$(arg simulate_perception)">
+        <origin xyz="-0.08 0.0 0.76" rpy="0 0 0"/>
+    </xacro:zed_camera>
+    <xacro:sensor_imu parent="chassis" prefix="zed_imu" topic_prefix="/camera">
+        <origin xyz="-0.08 0.0 0.76" rpy="0 0 0"/>
+    </xacro:sensor_imu>
+    <xacro:sensor_magnetometer parent="chassis" prefix="sbg">
+        <origin xyz="0.0 0.0 0.0" rpy="0 0 0"/>
+    </xacro:sensor_magnetometer>
+</robot>

File: eufs_sim/eufs_racecar/urdf/carro_enel_base.urdf.xacro (robot description, xacro)
@@ -1 +1,41 @@
-/home/gustavo/eufs_sim_teste/eufs_sim/eufs_racecar/urdf/carro_enel_base.urdf.xacro
+<?xml version="1.0"?>
+<!-- name enel ou carro_enel -->
+<robot name="carro_enel" xmlns:xacro="http://www.ros.org/wiki/xacro">
+  <xacro:macro name="carro_enel_base" params="chassis_mesh">
+    <xacro:property name="wheel_diameter" value="0.505"/>
+    <!-- BASE FOOTPRINT -->
+    <link name="base_footprint"/>
+    <joint name="chassis_joint" type="fixed">
+      <parent link="base_footprint"/>
+      <child link="chassis"/>
+      <origin xyz="0 0 ${wheel_diameter/2}"
+              rpy="0 0 0"/>
+      <axis xyz="1 0 0"/>
+    </joint>
+    <link name="chassis">
+      <visual>
+        <origin xyz="0 0 0" rpy="0 0 0" />
+        <geometry>
+          <mesh filename="${chassis_mesh}"/>
+        </geometry>
+      </visual>
+      <inertial>
+        <origin xyz="0 0 0" rpy="0 0 0" />
+        <mass value="140" />
+        <inertia
+            ixx="16.3"
+            ixy="0"
+            ixz="0"
+            iyy="33.6"
+            iyz="0"
+            izz="47.9" />
+      </inertial>
+      <collision>
+        <origin xyz="0 0 0" rpy="0 0 0" />
+        <geometry>
+          <mesh filename="${chassis_mesh}"/>
+        </geometry>
+      </collision>
+    </link>
+  </xacro:macro>
+</robot>

File: eufs_sim/eufs_racecar/urdf/carro_enel_wheels.urdf.xacro (robot description, xacro)
@@ -1 +1,117 @@
-/home/gustavo/eufs_sim_teste/eufs_sim/eufs_racecar/urdf/carro_enel_wheels.urdf.xacro
+<?xml version="1.0"?>
+<robot name="wheels" xmlns:xacro="http://www.ros.org/wiki/xacro">
+  <xacro:macro name="wheels"
+               params="chassis_width wheelbase">
+    <!-- ********** -->
+    <!-- Parameters -->
+    <!-- ********** -->
+    <xacro:property name="degrees_90" value="1.5708"/>
+    <xacro:property name="wheel_mass" value="10.0"/>
+    <xacro:property name="wheel_diameter" value="0.505"/>
+    <xacro:property name="wheel_width" value="0.2"/>
+    <xacro:property name="wheel_friction_mu1" value="2"/>
+    <xacro:property name="wheel_friction_mu2" value="2"/>
+    <xacro:property name="wheel_friction_kp" value="1e8"/>
+    <xacro:property name="steering_hinge_mass" value="1"/>
+    <!-- ***************** -->
+    <!-- Wheel description -->
+    <!-- ***************** -->
+    <xacro:macro name="wheel"
+                 params="lr_prefix fr_prefix">
+      <link name="${lr_prefix}_${fr_prefix}_wheel">
+        <inertial>
+          <origin xyz="0 0 0" rpy="0 0 0" />
+          <mass value="${wheel_mass}"/>
+          <inertia
+              ixx="0.3"
+              ixy="0"
+              ixz="0"
+              iyy="0.2"
+              iyz="0"
+              izz="0.2"   />
+        </inertial>
+        <visual>
+          <origin xyz="0 0 0" rpy="${degrees_90} 0 0"/>
+          <geometry>
+            <mesh filename="file://$(find eufs_racecar)/meshes/wheel_${lr_prefix}.dae"/>
+          </geometry>
+          <material name="tire_mat"/>
+        </visual>
+        <collision>
+          <origin xyz="0 0 0" rpy="${degrees_90} 0 0"/>
+          <geometry>
+            <cylinder radius="${wheel_diameter / 2}" length="${wheel_width}"/>
+          </geometry>
+        </collision>
+      </link>
+      <gazebo reference="${lr_prefix}_${fr_prefix}_wheel">
+        <material>Gazebo/Black</material>
+        <mu1>${wheel_friction_mu1}</mu1>
+        <mu2>${wheel_friction_mu2}</mu2>
+        <!-- <minDepth>0.005</minDepth> -->
+        <kp>${wheel_friction_kp}</kp>
+      </gazebo>
+    </xacro:macro>
+    <!-- ********************************* -->
+    <!-- Front and rear wheel descriptions -->
+    <!-- ********************************* -->
+    <!-- Description of how a front wheel is connected to the chassis -->
+    <xacro:macro name="front_wheel"
+                 params="lr_prefix lr_reflect">
+      <joint name="${lr_prefix}_steering_hinge_joint" type="revolute">
+        <origin xyz="${wheelbase / 2}
+                     ${lr_reflect * ((chassis_width - wheel_width) / 2)}
+                     0"
+                rpy="0 0 0"/>
+        <parent link="chassis"/>
+        <child link="${lr_prefix}_steering_hinge"/>
+        <axis xyz="0 0 1"/>
+        <limit lower="${config['input_ranges']['steering']['min']}" upper="${config['input_ranges']['steering']['max']}" effort="10000000" velocity="1000000"/>
+      </joint>
+      <link name="${lr_prefix}_steering_hinge">
+        <inertial>
+          <origin xyz="0 0 0" rpy="0 0 0" />
+          <mass value="${steering_hinge_mass}"/>
+          <inertia
+              ixx="0.04"
+              ixy="0.0"
+              ixz="0.0"
+              iyy="0.04"
+              iyz="0.0"
+              izz="0.04"   />
+        </inertial>
+      </link>
+      <joint name="front_${lr_prefix}_wheel_joint" type="continuous">
+        <origin xyz="0 0 0"
+                rpy="0 0 0"/>
+        <parent link="${lr_prefix}_steering_hinge"/>
+        <child link="${lr_prefix}_front_wheel"/>
+        <axis xyz="0 1 0"/>
+        <limit lower="0" upper="0" effort="10000000" velocity="1000000"/>
+      </joint>
+      <xacro:wheel lr_prefix="${lr_prefix}" fr_prefix="front"/>
+    </xacro:macro>
+    <!-- Description of how a rear wheel is connected to the chassis -->
+    <xacro:macro name="rear_wheel"
+                 params="lr_prefix lr_reflect">
+      <joint name="rear_${lr_prefix}_wheel_joint" type="continuous">
+        <origin xyz="${-1 * wheelbase / 2}
+                     ${lr_reflect * ((chassis_width - wheel_width) / 2)}
+                     0"
+                rpy="0 0 0"/>
+        <parent link="chassis"/>
+        <child link="${lr_prefix}_rear_wheel"/>
+        <axis xyz="0 1 0"/>
+        <limit lower="0" upper="0" effort="10000000" velocity="1000000"/>
+      </joint>
+      <xacro:wheel lr_prefix="${lr_prefix}" fr_prefix="rear"/>
+    </xacro:macro>
+    <!-- ************** -->
+    <!-- Add the wheels -->
+    <!-- ************** -->
+    <xacro:front_wheel lr_prefix="left" lr_reflect="1"/>
+    <xacro:front_wheel lr_prefix="right" lr_reflect="-1"/>
+    <xacro:rear_wheel lr_prefix="left" lr_reflect="1" />
+    <xacro:rear_wheel lr_prefix="right" lr_reflect="-1" />
+  </xacro:macro>
+</robot>
